File: Hardware/Reroute/SAMD21_Pro_RF_1W_reroute.brd (EAGLE design)
At the start: 53.3 x 40.6 mm, 138 parts, among them J10 AVR_SPI_PROG_3X2TESTPOINTS, J12 5.5x2.1mm Barrel, J13 U.FL, J7 PTH, J9 External On/Off, Q1 310mA/60V/1.6Ω, U1 MCP73831, U2 ADJ3.3, U3 3.3V, U4 ATSAMD21G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

Commit message: Started a re-route
Parts:
- removed D2: 3A/40V/500mV, SparkFun-DiscreteSemi:SMA-DIODE
- removed R11: 470, SparkFun-Resistors:0603
- removed R3: 10k, SparkFun-Resistors:0603
- removed R4: 787, SparkFun-Resistors:0603
- removed U2: ADJ3.3, SparkFun-IC-Power:SOT223
- added D5: 3A/10V/300mV, SAMD21_ProRF_1W:SOD-323
- D3: value 3A/40V/500mV -> 3A/10V/300mV; device SparkFun-DiscreteSemi:SMA-DIODE -> SAMD21_ProRF_1W:SOD-323
- R14: value 715 -> 750K
- moved R16 136.4 mm to (25.7, 18.4), turned to 270 degrees
- moved D3 131.9 mm to (21.5, 29.5), turned to 90 degrees
- moved R12 131.6 mm to (23.2, 17.5), turned to 180 degrees
- moved Q1 128.7 mm to (23.2, 19.7)
- moved JP1 112.3 mm to (26.8, 29.6), flipped to the bottom
- moved U3 112.0 mm to (26.8, 27.1), turned to 270 degrees
- moved J12 95.4 mm to (4.83, 13.2)
- moved R6 39.6 mm to (39.2, 9.27)
- moved U$70 26.1 mm to (49.4, 6.92), turned to 0 degrees
- moved U$72 25.3 mm to (49.4, 8.45), turned to 0 degrees
- moved R8 24.7 mm to (19.6, 12.2)
- moved U$65 24.7 mm to (49.4, 9.97), turned to 0 degrees
- moved U5 24.6 mm to (19.6, 8.48)
- moved D1 24.1 mm to (47.9, 6.92), turned to 180 degrees
- moved U$63 24.0 mm to (49.3, 11.5), turned to 0 degrees
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Connections:
- removed net N$10: C5.1, C7.+, C8.2, D3.A, R15.2, U7.2, U7.4
- removed net N$3: R11.2, U2.2, U2.4
- removed net N$4: D2.A, J12.VIN0
- removed net N$5: R11.1, R4.2, U2.1
- new net N$14: D5.A, R15.2, U7.2, U7.4
- net !RFM_CS5V: no longer R3.1
- net 3.3V: now also Q1.1
- net 5V: now also C5.1, C7.+, C8.2, D5.C; no longer R3.2
- net D10: now also U8.9; no longer U8.10
- net D11: now also U8.10; no longer U8.4
- net DIO05V: now also U8.13; no longer U8.12
- net DIO15V: now also U8.12; no longer U8.11
- net DIO25V: now also U8.11; no longer U8.17
- net GND: now also J12.GND; no longer R4.1
- net N$12: now also D3.A
- net RFM_INT: now also U8.8; no longer U8.9
- net RFM_RXEN: now also U8.7; no longer U8.8
- net RFM_RXEN5V: now also U8.14; no longer U8.13
- net RFM_TXEN: now also U8.4; no longer U8.7
- net RFM_TXEN5V: now also U8.17; no longer U8.14
- net VBATT: now also J12.VIN0; no longer D2.C
Routing:
- net 3.3V: track 234.0 -> 13.0 mm, vias 22 -> 0
- net GND: track 114.2 -> 32.8 mm, vias 28 -> 0
- net SDA: track 58.8 -> 0.00 mm, vias 2 -> 0
- net SCL: track 53.9 -> 0.00 mm, vias 3 -> 0
- net !RST: track 71.3 -> 17.7 mm, vias 4 -> 0
- net VBATT_LVL: track 44.7 -> 1.52 mm, vias 2 -> 0
- net CHARGE_STAT: track 35.9 -> 1.07 mm, vias 2 -> 1
- net RAW: track 63.0 -> 32.5 mm, vias 6 -> 2
- net SWDCLK: track 27.6 -> 0.00 mm, vias 4 -> 0
- net D10: track 31.2 -> 5.10 mm, vias 2 -> 0
- net RFM_INT: track 30.8 -> 5.34 mm, vias 2 -> 0
- net D8_!FLASH_CS: track 25.2 -> 0.00 mm, vias 4 -> 0
- net !RFM_CS: track 27.5 -> 3.65 mm, vias 2 -> 0
- net SCK: track 66.6 -> 43.2 mm, vias 5 -> 3
- net MISO: track 65.6 -> 42.4 mm, vias 6 -> 2
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