File: Hardware/Reroute/SAMD21_Pro_RF_1W_reroute.brd (EAGLE design)
At the start: 53.3 x 40.6 mm, 134 parts, among them J10 AVR_SPI_PROG_3X2TESTPOINTS, J12 5.5x2.1mm Barrel, J13 U.FL, J7 PTH, J9 External On/Off, Q1 310mA/60V/1.6Ω, U1 MCP73831, U3 3.3V, U4 ATSAMD21G, U5 4MB Flash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

Commit message: Finalized hardware
Parts:
- removed U$29: (no value), buzzard_labels (25):BATT25
- moved U$32 10.9 mm to (3.68, 5.59), flipped to the bottom, turned to 270 degrees
Routing:
- net 3.3V: track 113.3 -> 187.3 mm, vias 7 -> 13
- net USB_VCC: track 50.6 -> 97.3 mm, vias 4 -> 6
- net GND: track 33.1 -> 75.0 mm, vias 0 -> 20
- net !RST: track 52.5 -> 83.3 mm, vias 2 -> 5
- net 5V: track 59.3 -> 67.9 mm
- net N$14: track 20.1 -> 26.5 mm
- net !RFM_CS5V: track 33.2 -> 37.2 mm
- net CHARGE_STAT: track 78.2 -> 74.6 mm
- net SCK: track 71.8 -> 69.6 mm
- net RFM_RST: track 30.2 -> 32.0 mm
- net VBATT_LVL: track 53.1 -> 52.4 mm
- net RFM_TXEN5V: track 13.8 -> 14.5 mm
- net MOSI: track 72.4 -> 71.8 mm
- net RFM_RXEN5V: track 15.5 -> 15.0 mm
- net ANT: vias 0 -> 2
