File: Hardware/Reroute/SAMD21_Pro_RF_1W_reroute.sch (EAGLE design)
At the start: 70 parts, among them J10 AVR_SPI_PROG_3X2TESTPOINTS, J12 JST, J13 U.FL, J7 PTH, J9 External On/Off, U1 MCP73831, U2 ADJ3.3, U3 3.3V, U4 ATSAMD21G, U5 4MB Flash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

Commit message: Started a re-route
Parts:
- removed R11: 470, SparkFun-Resistors:470OHM-0603-1/10W-1%
- removed R3: 10k, SparkFun-Resistors:10KOHM-0603-1/10W-1%
- removed R4: 787, SparkFun-Resistors:787OHM-0603-1/10W-1%
- removed U2: ADJ3.3, SparkFun-IC-Power:V_REG_LM1117SOT223
- removed U9: TXB0108DQSR, SparkFun-IC-Comms:TXB0108
- added D3, D5: 3A/10V/300mV, SAMD21_ProRF_1W:DIODE-SCHOTTKY-BAT60A
- added Q1: 310mA/60V/1.6Ω, SparkFun-DiscreteSemi:MOSFET-NCH-2N7002PW
- added R12, R16: 10k, SparkFun-Resistors:10KOHM-0603-1/10W-1%
- F1: value 6V/0.75A -> 6V 0.5A; device SparkFun-Fuses:PPTC_THREE-QUARTER-AMP -> SparkFun-Fuses:PPTC_6V500MA
- J12: value JST -> 5.5x2.1mm Barrel; device SparkFun-Connectors:CONN_02-JST-2MM-SMT -> SparkFun-Connectors:POWER_JACKSMD
- R14: value 715 -> 750K; device SparkFun-Resistors:715OHM-0603-1/10W-1% -> SparkFun-Resistors:750KOHM-0603-1/10W-1%
Connections:
- removed net N$3: R11.2, U2.OUT, U2.OUT@1
- removed net N$5: R11.1, R4.2, U2.ADJ
- new net N$12: D3.A, F1.1, JP1.1
- new net N$14: D5.A, R15.2, U7.OUT, U7.OUT@1
- net !RFM_CS: now also Q1.S, R12.1; no longer U8.A4
- net !RFM_CS5V: now also Q1.D, R16.1; no longer R3.1, U8.B4
- net 3.3V: now also Q1.G, R12.2; no longer U9.OE, U9.VCCA
- net 5V: now also D3.C, D5.C, R16.2; no longer F1.1, JP1.1, R15.2, R3.2, U7.OUT, U7.OUT@1, U9.VCCB
- net D10: now also U8.A7; no longer U8.A8
- net D11: now also U8.A8; no longer U9.A4
- net DIO05V: now also U8.B6; no longer U8.B7
- net DIO15V: now also U8.B7; no longer U8.B8
- net DIO25V: now also U8.B8; no longer U9.B4
- net GND: now also J12.GND, J12.GNDBREAK; no longer J12.2, R4.1, U9.GND
- net RFM_INT: now also U8.A6; no longer U8.A7
- net RFM_RXEN: now also U8.A5; no longer U8.A6
- net RFM_RXEN5V: now also U8.B5; no longer U8.B6
- net RFM_TXEN: now also U8.A4; no longer U8.A5
- net RFM_TXEN5V: now also U8.B4; no longer U8.B5
- net VBATT: now also J12.PWR; no longer J12.1
Other:
- note added: "Solder this jumper if powering the board with VUSB and drawing more than 500 mA"
- note added: "VIN 7-15V"
- note removed: "Solder this jumper if powering the board with VUSB"
- moved on the sheet: C12, C13, C14, C5, C7, C8, J12, J7, J9, JP1, LED1, R1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
