File: Hardware/SAMD21_Pro_RF_1W.brd (EAGLE design)
At the start: 53.3 x 40.6 mm, 136 parts, among them J10 AVR_SPI_PROG_3X2TESTPOINTS, J12 5.5x2.1mm Barrel, J13 U.FL, J7 PTH, J9 External On/Off, Q1 310mA/60V/1.6Ω, U1 MCP73831, U3 3.3V, U4 ATSAMD21G, U5 4MB Flash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

Commit message: Started a re-route
Parts:
- removed D2: 3A/40V/500mV, SparkFun-DiscreteSemi:SMA-DIODE
- moved D5 163.8 mm to (14.0, 21.8)
- moved D3 161.4 mm to (14.0, 23.4)
- moved U3 136.9 mm to (67.4, 21.1)
- moved R16 131.1 mm to (18.0, 16.5), turned to 270 degrees
- moved R12 130.3 mm to (22.9, 16.3)
- moved Q1 123.5 mm to (19.8, 15.6)
- moved JP1 101.5 mm to (14.0, 24.9), flipped to the bottom
- moved J12 95.4 mm to (4.83, 13.2)
- moved C1 67.1 mm to (68.6, 29.2)
- moved R1 61.2 mm to (69.5, 14.0)
- moved R2 61.2 mm to (69.5, 11.4)
- moved U$29 11.5 mm to (-1.65, 7.49)
Connections:
- removed net N$4: D2.A, J12.VIN0
- net GND: now also J12.GND
- net VBATT: now also J12.VIN0; no longer D2.C
Routing:
- net N$14: track 0.31 -> 25.3 mm, vias 0 -> 2
- net !RFM_CS: track 27.5 -> 6.69 mm, vias 2 -> 1
- net 3.3V: track 234.0 -> 213.7 mm, vias 22 -> 21
- net GND: track 114.2 -> 96.6 mm, vias 28 -> 26
- net VBATT_LVL: track 44.7 -> 34.4 mm, vias 2 -> 1
- net VBATT: track 40.9 -> 50.7 mm
- net RAW: track 63.0 -> 54.9 mm, vias 6 -> 3
- net D11: track 27.9 -> 34.7 mm
- net D-: track 52.0 -> 45.3 mm, vias 6 -> 4
- net D+: track 50.1 -> 44.9 mm, vias 6 -> 4
- net 5V: track 56.8 -> 52.3 mm, vias 5 -> 6
- net N$12: track 0.00 -> 4.04 mm, vias 0 -> 1
- net DIO15V: track 32.6 -> 29.4 mm
- net RFM_RST: track 33.0 -> 30.2 mm, vias 1 -> 3
- net DIO05V: track 34.9 -> 33.2 mm
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
Commit message: Finalized hardware
Parts:
- removed R3: 10k, SparkFun-Resistors:0603
- removed U$29: (no value), buzzard_labels (25):BATT25
- moved C1 58.7 mm to (10.3, 22.5), turned to 180 degrees
- moved R2 56.7 mm to (13.7, 21.8), turned to 270 degrees
- moved R1 54.8 mm to (15.2, 21.8), turned to 90 degrees
- moved U3 41.1 mm to (26.8, 27.1), turned to 270 degrees
- moved R6 39.6 mm to (39.2, 9.27)
- moved U$70 26.1 mm to (49.4, 6.92), turned to 0 degrees
- moved U$72 25.3 mm to (49.4, 8.45), turned to 0 degrees
- moved R8 24.7 mm to (19.6, 12.2)
- moved U$65 24.7 mm to (49.4, 9.97), turned to 0 degrees
- moved U5 24.6 mm to (19.6, 8.48)
- moved D1 24.1 mm to (47.9, 6.92), turned to 180 degrees
- moved U$63 24.0 mm to (49.3, 11.5), turned to 0 degrees
- moved D6 23.3 mm to (47.9, 8.45), turned to 180 degrees
- moved D4 22.6 mm to (47.9, 9.97), turned to 180 degrees
- moved LED1 22.1 mm to (47.9, 11.5), turned to 0 degrees
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Connections:
- net !RFM_CS5V: no longer R3.1
- net 5V: no longer R3.2
- net D10: now also U8.9; no longer U8.10
- net D11: now also U8.10; no longer U8.4
- net DIO05V: now also U8.13; no longer U8.12
- net DIO15V: now also U8.12; no longer U8.11
- net DIO25V: now also U8.11; no longer U8.17
- net RFM_INT: now also U8.8; no longer U8.9
- net RFM_RXEN: now also U8.7; no longer U8.8
- net RFM_RXEN5V: now also U8.14; no longer U8.13
- net RFM_TXEN: now also U8.4; no longer U8.7
- net RFM_TXEN5V: now also U8.17; no longer U8.14
Routing:
- net CHARGE_STAT: track 35.9 -> 74.6 mm, vias 2 -> 4
- net 3.3V: track 213.7 -> 187.3 mm, vias 21 -> 13
- net RAW: track 54.9 -> 32.5 mm, vias 3 -> 2
- net !RFM_CS5V: track 14.9 -> 37.2 mm, vias 1 -> 3
- net USB_VCC: track 75.1 -> 97.3 mm
- net GND: track 96.6 -> 75.0 mm, vias 26 -> 20
- net MISO: track 65.6 -> 83.7 mm, vias 6 -> 5
- net VBATT_LVL: track 34.4 -> 52.4 mm, vias 1 -> 6
- net 5V: track 52.3 -> 67.9 mm, vias 6 -> 4
- net SWDCLK: track 27.6 -> 14.3 mm, vias 4 -> 1
- net DIO25V: track 9.38 -> 21.9 mm
- net TXO: track 34.1 -> 22.0 mm, vias 4 -> 1
- net !RST: track 71.3 -> 83.3 mm, vias 4 -> 5
- net MOSI: track 60.1 -> 71.8 mm, vias 6 -> 4
- net A4: track 34.1 -> 22.8 mm, vias 2 -> 1
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