File: Hardware/SAMD21_Pro_RF_1W.sch (EAGLE design)
At the start: 71 parts, among them J10 AVR_SPI_PROG_3X2TESTPOINTS, J12 5.5x2.1mm Barrel, J13 U.FL, J7 PTH, J9 External On/Off, Q1 310mA/60V/1.6Ω, U1 MCP73831, U3 3.3V, U4 ATSAMD21G, U5 4MB Flash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

Commit message: Finalized hardware
Parts:
- removed R3: 10k, SparkFun-Resistors:10KOHM-0603-1/10W-1%
Connections:
- net !RFM_CS5V: no longer R3.1
- net 5V: no longer R3.2
- net D10: now also U8.A7; no longer U8.A8
- net D11: now also U8.A8; no longer U8.A4
- net DIO05V: now also U8.B6; no longer U8.B7
- net DIO15V: now also U8.B7; no longer U8.B8
- net DIO25V: now also U8.B8; no longer U8.B4
- net RFM_INT: now also U8.A6; no longer U8.A7
- net RFM_RXEN: now also U8.A5; no longer U8.A6
- net RFM_RXEN5V: now also U8.B5; no longer U8.B6
- net RFM_TXEN: now also U8.A4; no longer U8.A5
- net RFM_TXEN5V: now also U8.B4; no longer U8.B5
Changed lines of the file:
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@@
 <part name="GND11" library="supply1" library_urn="urn:adsk.eagle:library:371" deviceset="GND" device=""/>
 <part name="U$34" library="SparkX" deviceset="SPARKX-LOGO" device="2"/>
-<part name="R3" library="SparkFun-Resistors" deviceset="10KOHM" device="-0603-1/10W-1%" value="10k"/>
 <part name="C5" library="SparkFun-Capacitors" deviceset="1.0UF" device="-0603-16V-10%" value="1.0uF"/>
 <part name="C7" library="SparkFun-Capacitors" deviceset="10UF-POLAR" device="-EIA3216-16V-10%(TANT)" value="10uF"/>
@@
 <part name="SUPPLY4" library="SparkFun-PowerSymbols" deviceset="5V" device=""/>
 <part name="P+7" library="SparkFun-PowerSymbols" deviceset="3.3V" device=""/>
-<part name="SUPPLY3" library="SparkFun-PowerSymbols" deviceset="5V" device=""/>
 <part name="J15" library="SparkFun-Connectors" deviceset="QWIIC_CONNECTOR" device="JS-1MM"/>
 <part name="P+13" library="SparkFun-PowerSymbols" deviceset="3.3V" device=""/>
@@
 <instance part="GND11" gate="1" x="198.12" y="10.16"/>
 <instance part="U$34" gate="G$1" x="391.16" y="40.64"/>
-<instance part="R3" gate="G$1" x="335.28" y="256.54" rot="R90"/>
 <instance part="C5" gate="G$1" x="274.32" y="254"/>
 <instance part="C7" gate="G$1" x="264.16" y="256.54"/>
@@
 <instance part="SUPPLY4" gate="G$1" x="345.44" y="193.04"/>
 <instance part="P+7" gate="G$1" x="314.96" y="193.04"/>
-<instance part="SUPPLY3" gate="G$1" x="335.28" y="264.16"/>
 <instance part="J15" gate="G$1" x="297.18" y="15.24" rot="MR0"/>
 <instance part="P+13" gate="G$1" x="287.02" y="22.86"/>
@@
 </segment>
 <segment>
-<pinref part="U8" gate="G$1" pin="A8"/>
-<wire x1="317.5" y1="165.1" x2="312.42" y2="165.1" width="0.1524" layer="91"/>
-<label x="312.42" y="165.1" size="1.27" layer="95" rot="R180" xref="yes"/>
+<label x="312.42" y="167.64" size="1.27" layer="95" rot="R180" xref="yes"/>
+<pinref part="U8" gate="G$1" pin="A7"/>
+<wire x1="317.5" y1="167.64" x2="312.42" y2="167.64" width="0.1524" layer="91"/>
 </segment>
 </net>
@@
 </segment>
 <segment>
-<pinref part="U8" gate="G$1" pin="A4"/>
-<wire x1="317.5" y1="180.34" x2="312.42" y2="180.34" width="0.1524" layer="91"/>
-<label x="312.42" y="180.34" size="1.27" layer="95" rot="R180" xref="yes"/>
+<pinref part="U8" gate="G$1" pin="A8"/>
+<wire x1="317.5" y1="165.1" x2="312.42" y2="165.1" width="0.1524" layer="91"/>
+<label x="312.42" y="165.1" size="1.27" layer="95" rot="R180" xref="yes"/>
 </segment>
 </net>
@@
 </segment>
 <segment>
-<pinref part="U8" gate="G$1" pin="A7"/>
-<wire x1="317.5" y1="167.64" x2="312.42" y2="167.64" width="0.1524" layer="91"/>
-<label x="312.42" y="167.64" size="1.27" layer="95" rot="R180" xref="yes"/>
+<label x="312.42" y="170.18" size="1.27" layer="95" rot="R180" xref="yes"/>
+<pinref part="U8" gate="G$1" pin="A6"/>
+<wire x1="317.5" y1="170.18" x2="312.42" y2="170.18" width="0.1524" layer="91"/>
 </segment>
 </net>
@@
 <wire x1="345.44" y1="177.8" x2="345.44" y2="193.04" width="0.1524" layer="91"/>
 <pinref part="SUPPLY4" gate="G$1" pin="5V"/>
-</segment>
-<segment>
-<pinref part="R3" gate="G$1" pin="2"/>
-<wire x1="335.28" y1="264.16" x2="335.28" y2="261.62" width="0.1524" layer="91"/>
-<pinref part="SUPPLY3" gate="G$1" pin="5V"/>
 </segment>
 <segment>
@@
 </segment>
 <segment>
-<pinref part="U8" gate="G$1" pin="A6"/>
-<wire x1="317.5" y1="170.18" x2="312.42" y2="170.18" width="0.1524" layer="91"/>
-<label x="312.42" y="170.18" size="1.27" layer="95" rot="R180" xref="yes"/>
+<label x="312.42" y="172.72" size="1.27" layer="95" rot="R180" xref="yes"/>
+<pinref part="U8" gate="G$1" pin="A5"/>
+<wire x1="317.5" y1="172.72" x2="312.42" y2="172.72" width="0.1524" layer="91"/>
 </segment>
 </net>
@@
 </segment>
 <segment>
-<pinref part="U8" gate="G$1" pin="A5"/>
-<wire x1="317.5" y1="172.72" x2="312.42" y2="172.72" width="0.1524" layer="91"/>
-<label x="312.42" y="172.72" size="1.27" layer="95" rot="R180" xref="yes"/>
+<label x="312.42" y="180.34" size="1.27" layer="95" rot="R180" xref="yes"/>
+<pinref part="U8" gate="G$1" pin="A4"/>
+<wire x1="317.5" y1="180.34" x2="312.42" y2="180.34" width="0.1524" layer="91"/>
 </segment>
 </net>
@@
 <segment>
 <pinref part="U6" gate="G$1" pin="SCK"/>
-<wire x1="337.82" y1="236.22" x2="332.74" y2="236.22" width="0.1524" layer="91"/>
-<label x="332.74" y="236.22" size="1.27" layer="95" rot="R180" xref="yes"/>
+<wire x1="337.82" y1="236.22" x2="335.28" y2="236.22" width="0.1524" layer="91"/>
+<label x="335.28" y="236.22" size="1.27" layer="95" rot="R180" xref="yes"/>
 </segment>
 </net>
@@
 <segment>
 <pinref part="U6" gate="G$1" pin="MOSI"/>
-<wire x1="337.82" y1="241.3" x2="332.74" y2="241.3" width="0.1524" layer="91"/>
-<label x="332.74" y="241.3" size="1.27" layer="95" rot="R180" xref="yes"/>
+<wire x1="337.82" y1="241.3" x2="335.28" y2="241.3" width="0.1524" layer="91"/>
+<label x="335.28" y="241.3" size="1.27" layer="95" rot="R180" xref="yes"/>
 </segment>
 <segment>
@@
 <segment>
 <pinref part="U6" gate="G$1" pin="MISO"/>
-<wire x1="337.82" y1="238.76" x2="332.74" y2="238.76" width="0.1524" layer="91"/>
-<label x="332.74" y="238.76" size="1.27" layer="95" rot="R180" xref="yes"/>
+<wire x1="337.82" y1="238.76" x2="335.28" y2="238.76" width="0.1524" layer="91"/>
+<label x="335.28" y="238.76" size="1.27" layer="95" rot="R180" xref="yes"/>
 </segment>
 <segment>
@@
 <segment>
 <pinref part="U6" gate="G$1" pin="!NSS"/>
+<label x="335.28" y="243.84" size="1.27" layer="95" rot="R180" xref="yes"/>
 <wire x1="337.82" y1="243.84" x2="335.28" y2="243.84" width="0.1524" layer="91"/>
-<label x="332.74" y="243.84" size="1.27" layer="95" rot="R180" xref="yes"/>
-<pinref part="R3" gate="G$1" pin="1"/>
-<wire x1="335.28" y1="243.84" x2="332.74" y2="243.84" width="0.1524" layer="91"/>
-<wire x1="335.28" y1="251.46" x2="335.28" y2="243.84" width="0.1524" layer="91"/>
-<junction x="335.28" y="243.84"/>
 </segment>
 <segment>
@@
 <net name="RFM_TXEN5V" class="0">
 <segment>
+<label x="347.98" y="180.34" size="1.27" layer="95" xref="yes"/>
+<pinref part="U8" gate="G$1" pin="B4"/>
+<wire x1="342.9" y1="180.34" x2="347.98" y2="180.34" width="0.1524" layer="91"/>
+</segment>
+<segment>
+<pinref part="U6" gate="G$1" pin="TXEN"/>
+<wire x1="337.82" y1="246.38" x2="335.28" y2="246.38" width="0.1524" layer="91"/>
+<label x="335.28" y="246.38" size="1.27" layer="95" rot="R180" xref="yes"/>
+</segment>
+</net>
+<net name="RFM_RXEN5V" class="0">
+<segment>
+<label x="347.98" y="172.72" size="1.27" layer="95" xref="yes"/>
 <pinref part="U8" gate="G$1" pin="B5"/>
 <wire x1="342.9" y1="172.72" x2="347.98" y2="172.72" width="0.1524" layer="91"/>
-<label x="347.98" y="172.72" size="1.27" layer="95" xref="yes"/>
-</segment>
-<segment>
-<pinref part="U6" gate="G$1" pin="TXEN"/>
-<wire x1="337.82" y1="246.38" x2="332.74" y2="246.38" width="0.1524" layer="91"/>
-<label x="332.74" y="246.38" size="1.27" layer="95" rot="R180" xref="yes"/>
-</segment>
-</net>
-<net name="RFM_RXEN5V" class="0">
-<segment>
+</segment>
+<segment>
+<pinref part="U6" gate="G$1" pin="RXEN"/>
+<wire x1="337.82" y1="248.92" x2="335.28" y2="248.92" width="0.1524" layer="91"/>
+<label x="335.28" y="248.92" size="1.27" layer="95" rot="R180" xref="yes"/>
+</segment>
+</net>
+<net name="DIO05V" class="0">
+<segment>
+<label x="347.98" y="170.18" size="1.27" layer="95" xref="yes"/>
 <pinref part="U8" gate="G$1" pin="B6"/>
 <wire x1="342.9" y1="170.18" x2="347.98" y2="170.18" width="0.1524" layer="91"/>
-<label x="347.98" y="170.18" size="1.27" layer="95" xref="yes"/>
-</segment>
-<segment>
-<pinref part="U6" gate="G$1" pin="RXEN"/>
-<wire x1="337.82" y1="248.92" x2="332.74" y2="248.92" width="0.1524" layer="91"/>
-<label x="332.74" y="248.92" size="1.27" layer="95" rot="R180" xref="yes"/>
-</segment>
-</net>
-<net name="DIO05V" class="0">
-<segment>
-<pinref part="U8" gate="G$1" pin="B7"/>
-<wire x1="342.9" y1="167.64" x2="347.98" y2="167.64" width="0.1524" layer="91"/>
-<label x="347.98" y="167.64" size="1.27" layer="95" xref="yes"/>
 </segment>
 <segment>
@@
 <net name="DIO15V" class="0">
 <segment>
+<label x="347.98" y="167.64" size="1.27" layer="95" xref="yes"/>
+<pinref part="U8" gate="G$1" pin="B7"/>
+<wire x1="342.9" y1="167.64" x2="347.98" y2="167.64" width="0.1524" layer="91"/>
+</segment>
+<segment>
+<pinref part="U6" gate="G$1" pin="DIO1"/>
+<wire x1="368.3" y1="236.22" x2="365.76" y2="236.22" width="0.1524" layer="91"/>
+<label x="368.3" y="236.22" size="1.27" layer="95" xref="yes"/>
+</segment>
+</net>
+<net name="DIO25V" class="0">
+<segment>
+<pinref part="U6" gate="G$1" pin="DIO2"/>
+<wire x1="368.3" y1="238.76" x2="365.76" y2="238.76" width="0.1524" layer="91"/>
+<label x="368.3" y="238.76" size="1.27" layer="95" xref="yes"/>
+</segment>
+<segment>
 <pinref part="U8" gate="G$1" pin="B8"/>
 <wire x1="342.9" y1="165.1" x2="347.98" y2="165.1" width="0.1524" layer="91"/>
 <label x="347.98" y="165.1" size="1.27" layer="95" xref="yes"/>
 </segment>
-<segment>
-<pinref part="U6" gate="G$1" pin="DIO1"/>
-<wire x1="368.3" y1="236.22" x2="365.76" y2="236.22" width="0.1524" layer="91"/>
-<label x="368.3" y="236.22" size="1.27" layer="95" xref="yes"/>
-</segment>
-</net>
-<net name="DIO25V" class="0">
-<segment>
-<pinref part="U6" gate="G$1" pin="DIO2"/>
-<wire x1="368.3" y1="238.76" x2="365.76" y2="238.76" width="0.1524" layer="91"/>
-<label x="368.3" y="238.76" size="1.27" layer="95" xref="yes"/>
-</segment>
-<segment>
-<pinref part="U8" gate="G$1" pin="B4"/>
-<wire x1="342.9" y1="180.34" x2="347.98" y2="180.34" width="0.1524" layer="91"/>
-<label x="347.98" y="180.34" size="1.27" layer="95" xref="yes"/>
-</segment>
-</net>
+</net>
