File: Hardware/Production/SAMD21_Pro_RF_1W-Panel.brd (EAGLE design)
At the start: 53.3 x 40.6 mm, 134 parts, among them J10 AVR_SPI_PROG_3X2TESTPOINTS, J12 5.5x2.1mm Barrel, J13 U.FL, J7 PTH, J9 External On/Off, Q1 310mA/60V/1.6Ω, U1 MCP73831, U3 3.3V, U4 ATSAMD21G, U5 4MB Flash, U6 E19-915MS1W, U7 ADJ5, U8 TXB0108DQSR, Y1 32.768kHz

Commit message: Finalizing
Parts:
- removed FRAME2: FRAME-LEDGER, SparkFun-Aesthetics:CREATIVE_COMMONS
- added C16, C19, C29, C31, C34, C44, C46, C49, C59: 10uF, SparkFun-Capacitors:EIA3216
- added C17, C20, C24, C25, C26, C27, C30, C32, C35, C39, C40, C41, C42, C45, C47, C50, C54, C55, C56, C57, C60: 0.1uF, SparkFun-Capacitors:0603
- added C18, C28, C33, C43, C48, C58: 1.0uF, SparkFun-Capacitors:0603
- added C21, C36, C51: 4.7uF, SparkFun-Capacitors:0603
- added C22, C23, C37, C38, C52, C53: 15pF, SparkFun-Capacitors:0603
- added D10, D14, D15, D19, D20, D9: 3A/10V/300mV, SAMD21_ProRF_1W:SOD-323
- added D11, D16, D2: Green, SparkFun-LED:LED-0603
- added D12, D17, D7: BLUE, SparkFun-LED:LED-0603
- added D13, D18, D8: Yellow, SparkFun-LED:LED-0603
- added E$1, E$2, E$3, E$4: (no value), SparkFun-Aesthetics:FIDUCIAL-1X2
- added E$5, E$6: (no value), SparkFun-Retired:FIDUCIAL-1.5X3
- added F2, F3, F4: 6V 0.5A, SparkFun-Fuses:0805
- added FD10, FD11, FD12, FD13, FD14, FD15, FD16, FD5, FD6, FD7, FD8, FD9: FIDUCIAL1X2, SparkFun-Aesthetics:FIDUCIAL-1X2
- added J14, J29, J43: (no value), SparkFun-Connectors:USB-MICROB-PTH-MILL
- added J16, J30, J44: PTH, SparkFun-Connectors:1X02_NO_SILK
- added J17, J31, J45: (no value), SparkFun-Connectors:1X02_NO_SILK
- added J18, J32, J46: External On/Off, SparkFun-Connectors:1X02_NO_SILK
- added J19, J20, J33, J34, J47, J48: (no value), SparkFun-Connectors:1X10_NO_SILK
- added J21, J23, J35, J37, J49, J51: (no value), SparkFun-Connectors:1X09_NO_SILK
- added J22, J36, J50: AVR_SPI_PROG_3X2TESTPOINTS, SparkFun-Connectors:2X3_TEST_POINTS
- added J24, J38, J52: (no value), SparkFun-Connectors:1X01_NO_SILK
- added J25, J39, J53: U.FL, SparkFun-Connectors:U.FL
- added J26, J27, J40, J41, J54, J55: (no value), SparkFun-Connectors:1X04_1MM_RA
- added J28, J42, J56: 5.5x2.1mm Barrel, SparkFun-Connectors:POWER_JACK_SMD
- added JP2, JP3, JP4: FuseBypass, SparkFun-Jumpers:SMT-JUMPER_2_NO_SILK
- added L2, L3, L4: (no value), SparkFun-Coils:0603
- added LED2, LED3, LED4: RED, SparkFun-LED:LED-0603
- added LOGO2, LOGO3, LOGO4: OSHW-LOGOMINI, SparkFun-Aesthetics:OSHW-LOGO-MINI
- added Q2, Q3, Q4: 310mA/60V/1.6Ω, SparkFun-DiscreteSemi:SOT323
- added R11, R29, R42: 2.0k, SparkFun-Resistors:0603
- added R17, R20, R21, R22, R25, R26, R30, R33, R34, R35, R38, R39, R43, R46, R47, R48, R51, R52: 10k, SparkFun-Resistors:0603
- added R18, R19, R27, R28, R3, R31, R32, R4, R40, R41, R44, R45: 1k, SparkFun-Resistors:0603
- added R23, R36, R49: 750K, SparkFun-Resistors:0603
- added R24, R37, R50: 240, SparkFun-Resistors:0603
- added S2, S5, S7: Power, SparkFun-Switches:SWITCH_SPST_SMD_A
- added S4, S6, S8: (no value), SparkFun-Switches:TACTILE_SWITCH_SMD_RIGHT_ANGLE
- added U$100, U$165, U$230: (no value), buzzard_labels (8):RX7
- added U$101, U$107, U$166, U$172, U$231, U$237: (no value), buzzard_labels (8):RX2
- added U$102, U$167, U$232: (no value), buzzard_labels (9):CHG1
- added U$103, U$168, U$233: (no value), buzzard_labels (25):D514
- added U$104, U$105, U$169, U$170, U$234, U$235: (no value), buzzard_labels (10):D90
- added U$106, U$140, U$147, U$161, U$171, U$205, U$212, U$226, U$236, U$74, U$82, U$96: (no value), buzzard_labels (25):GND0
- added U$108, U$163, U$173, U$228, U$238, U$98: (no value), buzzard_labels (8):TX3
- added U$109, U$113, U$174, U$178, U$239, U$243: (no value), D2:D20
- added U$110, U$114, U$175, U$179, U$240, U$244: (no value), D3:D30
- added U$111, U$115, U$176, U$180, U$241, U$245: (no value), D4:D40
- added U$112, U$177, U$242: (no value), D5:D50
- added U$116, U$181, U$246: SPARKX-LOGO2, SparkX:SPARKX-TINY
- added U$117, U$182, U$247: (no value), Labels:QWIIC-LOGO-MEDIUM
- added U$118, U$183, U$248: (no value), SparkX:SPARKX-MEDIUM
- added U$119, U$184, U$249: (no value), SparkFun-Aesthetics:OSHW-LOGO-MINI
- added U$120, U$185, U$250: (no value), buzzard_labels:SAMD21_PRORF_1W5
- added U$121, U$122, U$186, U$187, U$251, U$252: (no value), buzzard_labels:VUSB7
- added U$123, U$124, U$188, U$189, U$253, U$254: (no value), buzzard_labels:SWITCH6
- added U$125, U$126, U$129, U$130, U$190, U$191, U$194, U$195, U$255, U$256, U$259, U$260: (no value), Labels:QWIIC-TEXT-04
- added U$127, U$192, U$257: (no value), buzzard_labels:7#15V0
- added U$128, U$193, U$258: (no value), buzzard_labels:SOLDER_TO_BYPASS_VUSB_FUSE1
- added U$131, U$150, U$196, U$215, U$85: (no value), buzzard_labels (25):A43
- added U$132, U$151, U$197, U$216, U$58, U$86: (no value), buzzard_labels (25):A34
- added U$133, U$152, U$198, U$217, U$59, U$87: (no value), buzzard_labels (25):A25
- added U$134, U$153, U$199, U$218, U$60, U$88: (no value), buzzard_labels (25):A16
- added U$135, U$154, U$200, U$219, U$64, U$89: (no value), buzzard_labels (25):A07
- added U$136, U$155, U$201, U$220, U$66, U$90: (no value), buzzard_labels (25):MISO8
- added U$137, U$156, U$202, U$221, U$67, U$91: (no value), buzzard_labels (25):MOSI9
- added U$138, U$157, U$203, U$222, U$68, U$92: (no value), buzzard_labels (25):SCK10
- added U$139, U$158, U$204, U$223, U$71, U$93: (no value), buzzard_labels (25):ANT11
- added U$141, U$144, U$146, U$149, U$206, U$209, U$211, U$214, U$75, U$78, U$80, U$84: (no value), buzzard_labels (25):RST2
- added U$142, U$160, U$207, U$225, U$76, U$95: (no value), buzzard_labels (25):3V320
- added U$143, U$159, U$208, U$224, U$77, U$94: (no value), buzzard_labels (25):RAW21
- added U$145, U$210, U$79: (no value), buzzard_labels (25):BATT25
- added U$148, U$213, U$83: (no value), buzzard_labels (28):ON#OFF0
- added U$162, U$227, U$97: (no value), Labels:PWR-()-03
- added U$164, U$229, U$99: (no value), buzzard_labels (8):TX6
- added U10, U17, U24: ATSAMD21G, temp:QFN-48_NO_EXPOSED_PAD
- added U11, U18, U25: ADJ5, SparkFun-IC-Power:SOT223
- added U12, U19, U26: E19-915MS1W, SAMD21_ProRF_1W:E19-915MS1W
- added U13, U20, U27: TXB0108DQSR, SparkFun-IC-Comms:UFDFN-20
- added U14, U21, U28: 3.3V, SparkFun-IC-Power:SOT23-5
- added U15, U2, U22: MCP73831, SparkFun-IC-Power:SOT23-5
- added U16, U23, U9: 4MB Flash, SparkFun-IC-Memory:SO08
- added Y2, Y3, Y4: 32.768kHz, SparkFun-Clocks:CRYSTAL-SMD-3.2X1.5MM
- U$26: value SPECIAL_INSTRUCTIONS-ORDERING -> (none); device SparkFun-Aesthetics:ORDERING_INSTRUCTIONS -> buzzard_labels (25):A43
- moved U$26 129.5 mm to (85.5, 35.3)
Connections:
- new net !RFM_CS1: Q2.2, R25.1, U10.28
- new net !RFM_CS2: Q3.2, R38.1, U17.28
- new net !RFM_CS3: Q4.2, R51.1, U24.28
- new net !RFM_CS5V1: Q2.3, R26.1, U12.P$15
- new net !RFM_CS5V2: Q3.3, R39.1, U19.P$15
- new net !RFM_CS5V3: Q4.3, R52.1, U26.P$15
- new net !RST1: J19.8, J22.5, R17.1, S4.1, U10.40
- new net !RST2: J33.8, J36.5, R30.1, S6.1, U17.40
- new net !RST3: J47.8, J50.5, R43.1, S8.1, U24.40
- new net 3.3V1: C18.1, C19.+, C20.2, C24.2, C25.2, C27.2, D2.A, D8.A, J19.2, J22.2, J26.2, J27.2, L2.1, Q2.1, R17.2, R22.2, R25.2, R4.2, U10.17, U10.36, U10.43, U10.44, U13.5, U13.6, U14.5, U9.3, U9.7, U9.8
- new net 3.3V2: C33.1, C34.+, C35.2, C39.2, C40.2, C42.2, D11.A, D13.A, J33.2, J36.2, J40.2, J41.2, L3.1, Q3.1, R28.2, R30.2, R35.2, R38.2, U16.3, U16.7, U16.8, U17.17, U17.36, U17.43, U17.44, U20.5, U20.6, U21.5
- new net 3.3V3: C48.1, C49.+, C50.2, C54.2, C55.2, C57.2, D16.A, D18.A, J47.2, J50.2, J54.2, J55.2, L4.1, Q4.1, R41.2, R43.2, R48.2, R51.2, U23.3, U23.7, U23.8, U24.17, U24.36, U24.43, U24.44, U27.5, U27.6, U28.5
- new net 5V1: C28.1, C29.+, C30.2, D10.C, D9.C, R26.2, U12.P$11, U13.16, U14.1, U14.3
- new net 5V2: C43.1, C44.+, C45.2, D14.C, D15.C, R39.2, U19.P$11, U20.16, U21.1, U21.3
- new net 5V3: C58.1, C59.+, C60.2, D19.C, D20.C, R52.2, U26.P$11, U27.16, U28.1, U28.3
- new net A10: J37.9, U17.3
- new net A11: J37.8, U17.7
- new net A12: J37.7, U17.8
- new net A13: J37.6, U17.9
- new net A14: J37.5, U17.10
- new net A15: J51.9, U24.3
- new net A16: J51.8, U24.7
- new net A17: J51.7, U24.8
- new net A18: J51.6, U24.9
- new net A19: J51.5, U24.10
- new net A5: J23.9, U10.3
- new net A6: J23.8, U10.7
- new net A7: J23.7, U10.8
- new net A8: J23.6, U10.9
- new net A9: J23.5, U10.10
- new net ANT1: J24.1, J25.FEED, U12.P$19
- new net ANT2: J38.1, J39.FEED, U19.P$19
- new net ANT3: J52.1, J53.FEED, U26.P$19
- new net CHARGE_STAT1: R19.1, U2.1
- new net CHARGE_STAT2: R32.1, U15.1
- new net CHARGE_STAT3: R45.1, U22.1
- new net D+1: J14.D+, U10.34
- new net D+2: J29.D+, U17.34
- new net D+3: J43.D+, U24.34
- new net D-1: J14.D-, U10.33
- new net D-2: J29.D-, U17.33
- new net D-3: J43.D-, U24.33
- new net D1: J19.4, U10.13
- new net D12: J19.5, U10.14
- new net D13: J19.7, U10.24
- new net D14: J19.3, U10.12
- new net D15: J33.4, U17.13
- new net D16: U17.27, U20.9
- new net D17: U17.25, U20.10
- new net D18: J33.6, U17.23
- new net D19: J33.5, U17.14
- new net D20: J33.7, U17.24
- new net D21: J33.3, U17.12
- new net D22: J47.4, U24.13
- new net D23: U24.27, U27.9
- new net D24: U24.25, U27.10
- new net D25: J47.6, U24.23
- new net D26: J47.5, U24.14
- new net D27: J47.7, U24.24
- new net D28: J47.3, U24.12
- new net D6: U10.27, U13.9
- new net D7: U10.25, U13.10
- new net D8: J19.6, U10.23
- new net D8_!FLASH_CS1: R22.1, U10.11, U9.1
- new net D8_!FLASH_CS2: R35.1, U16.1, U17.11
- new net D8_!FLASH_CS3: R48.1, U23.1, U24.11
- new net DIO05V1: U12.P$7, U13.13
- new net DIO05V2: U19.P$7, U20.13
- new net DIO05V3: U26.P$7, U27.13
- new net DIO15V1: U12.P$6, U13.12
- new net DIO15V2: U19.P$6, U20.12
- new net DIO15V3: U26.P$6, U27.12
- new net DIO25V1: U12.P$5, U13.11
- new net DIO25V2: U19.P$5, U20.11
- new net DIO25V3: U26.P$5, U27.11
- new net GND1: C16.-, C17.1, C18.2, C19.-, C20.1, C21.2, C22.1, C23.1, C24.1, C25.1, C26.1, C27.1, C28.2, C29.-, C30.1, J14.GND, J16.1, J17.1, J20.1, J20.10, J20.2, J20.3, J20.4, J20.5, J20.6, J20.7, J20.8, J20.9, J21.1, J21.2, J21.3, J21.4, J21.5, J21.6, J21.7, J21.8, J21.9, J22.6, J23.1, J25.1, J25.2, J26.1, J27.1, J28.GND, J28.P$4, LED2.C, R11.2, R21.1, R23.1, S4.2, U10.18, U10.35, U10.42, U10.5, U12.P$1, U12.P$10, U12.P$18, U12.P$20, U12.P$21, U12.P$22, U12.P$9, U13.15, U14.2, U2.2, U9.4
- new net GND2: C31.-, C32.1, C33.2, C34.-, C35.1, C36.2, C37.1, C38.1, C39.1, C40.1, C41.1, C42.1, C43.2, C44.-, C45.1, J29.GND, J30.1, J31.1, J34.1, J34.10, J34.2, J34.3, J34.4, J34.5, J34.6, J34.7, J34.8, J34.9, J35.1, J35.2, J35.3, J35.4, J35.5, J35.6, J35.7, J35.8, J35.9, J36.6, J37.1, J39.1, J39.2, J40.1, J41.1, J42.GND, J42.P$4, LED3.C, R29.2, R34.1, R36.1, S6.2, U15.2, U16.4, U17.18, U17.35, U17.42, U17.5, U19.P$1, U19.P$10, U19.P$18, U19.P$20, U19.P$21, U19.P$22, U19.P$9, U20.15, U21.2
- new net GND3: C46.-, C47.1, C48.2, C49.-, C50.1, C51.2, C52.1, C53.1, C54.1, C55.1, C56.1, C57.1, C58.2, C59.-, C60.1, J43.GND, J44.1, J45.1, J48.1, J48.10, J48.2, J48.3, J48.4, J48.5, J48.6, J48.7, J48.8, J48.9, J49.1, J49.2, J49.3, J49.4, J49.5, J49.6, J49.7, J49.8, J49.9, J50.6, J51.1, J53.1, J53.2, J54.1, J55.1, J56.GND, J56.P$4, LED4.C, R42.2, R47.1, R49.1, S8.2, U22.2, U23.4, U24.18, U24.35, U24.42, U24.5, U26.P$1, U26.P$10, U26.P$18, U26.P$20, U26.P$21, U26.P$22, U26.P$9, U27.15, U28.2
- new net MISO1: J22.1, J23.2, U10.21, U13.2, U9.2
- new net MISO2: J36.1, J37.2, U16.2, U17.21, U20.2
- new net MISO3: J50.1, J51.2, U23.2, U24.21, U27.2
- new net MISO5V1: U12.P$13, U13.19
- new net MISO5V2: U19.P$13, U20.19
- new net MISO5V3: U26.P$13, U27.19
- new net MOSI1: J23.3, U10.19, U13.3, U9.5
- new net MOSI2: J37.3, U16.5, U17.19, U20.3
- new net MOSI3: J51.3, U23.5, U24.19, U27.3
- new net MOSI5V1: U12.P$14, U13.18
- new net MOSI5V2: U19.P$14, U20.18
- new net MOSI5V3: U26.P$14, U27.18
- new net N$10: LED2.A, R4.1
- new net N$15: D8.C, R3.2
- new net N$16: D2.C, R18.2
- new net N$17: C22.2, U10.1, Y2.P$2
- new net N$18: C23.2, U10.2, Y2.P$1
- new net N$19: R23.2, R24.1, U11.1
- new net N$20: D9.A, F2.1, JP2.1
- new net N$21: D10.A, R24.2, U11.2, U11.4
- new net N$22: J32.2, S5.1
- new net N$23: R29.1, U15.5
- new net N$24: D12.C, R32.2
- new net N$25: LED3.A, R28.1
- new net N$26: D13.C, R27.2
- new net N$27: D11.C, R31.2
- new net N$28: C37.2, U17.1, Y3.P$2
- new net N$29: C38.2, U17.2, Y3.P$1
- new net N$3: J18.2, S2.1
- new net N$30: R36.2, R37.1, U18.1
- new net N$31: D14.A, F3.1, JP3.1
- new net N$32: D15.A, R37.2, U18.2, U18.4
- new net N$33: J46.2, S7.1
- new net N$34: R42.1, U22.5
- new net N$35: D17.C, R45.2
- new net N$36: LED4.A, R41.1
- new net N$37: D18.C, R40.2
- new net N$39: D16.C, R44.2
- new net N$4: R11.1, U2.5
- new net N$40: C52.2, U24.1, Y4.P$2
- new net N$41: C53.2, U24.2, Y4.P$1
- new net N$42: R49.2, R50.1, U25.1
- new net N$43: D19.A, F4.1, JP4.1
- new net N$44: D20.A, R50.2, U25.2, U25.4
- new net N$5: D7.C, R19.2
- new net RAW1: J18.1, J19.1, S2.2, U11.3
- new net RAW2: J32.1, J33.1, S5.2, U18.3
- new net RAW3: J46.1, J47.1, S7.2, U25.3
- new net RFM_INT1: U10.29, U13.8
- new net RFM_INT2: U17.29, U20.8
- new net RFM_INT3: U24.29, U27.8
- new net RFM_RST1: U10.26, U12.P$8
- new net RFM_RST2: U17.26, U19.P$8
- new net RFM_RST3: U24.26, U26.P$8
- new net RFM_RXEN1: U10.38, U13.7
- new net RFM_RXEN2: U17.38, U20.7
- new net RFM_RXEN3: U24.38, U27.7
- new net RFM_RXEN5V1: U12.P$17, U13.14
- new net RFM_RXEN5V2: U19.P$17, U20.14
- new net RFM_RXEN5V3: U26.P$17, U27.14
- new net RFM_TXEN1: U10.37, U13.4
- new net RFM_TXEN2: U17.37, U20.4
- new net RFM_TXEN3: U24.37, U27.4
- new net RFM_TXEN5V1: U12.P$16, U13.17
- new net RFM_TXEN5V2: U19.P$16, U20.17
- new net RFM_TXEN5V3: U26.P$16, U27.17
- new net RXI1: J19.10, U10.16
- new net RXI2: J33.10, U17.16
- new net RXI3: J47.10, U24.16
- new net RX_LED1: R3.1, U10.48
- new net RX_LED2: R27.1, U17.48
- new net RX_LED3: R40.1, U24.48
- new net SCK1: J23.4, U10.20, U13.1, U9.6
- new net SCK2: J37.4, U16.6, U17.20, U20.1
- new net SCK3: J51.4, U23.6, U24.20, U27.1
- new net SCK5V1: U12.P$12, U13.20
- new net SCK5V2: U19.P$12, U20.20
- new net SCK5V3: U26.P$12, U27.20
- new net SCL1: J26.4, J27.4, U10.32
- new net SCL2: J40.4, J41.4, U17.32
- new net SCL3: J54.4, J55.4, U24.32
- new net SDA1: J26.3, J27.3, U10.31
- new net SDA2: J40.3, J41.3, U17.31
- new net SDA3: J54.3, J55.3, U24.31
- new net SHLD1: J14.SHIELD, J14.SHIELD10, J14.SHIELD2, J14.SHIELD3, J14.SHIELD4, J14.SHIELD5, J14.SHIELD6, J14.SHIELD7, J14.SHIELD8, J14.SHIELD9
- new net SHLD2: J29.SHIELD, J29.SHIELD10, J29.SHIELD2, J29.SHIELD3, J29.SHIELD4, J29.SHIELD5, J29.SHIELD6, J29.SHIELD7, J29.SHIELD8, J29.SHIELD9
- new net SHLD3: J43.SHIELD, J43.SHIELD10, J43.SHIELD2, J43.SHIELD3, J43.SHIELD4, J43.SHIELD5, J43.SHIELD6, J43.SHIELD7, J43.SHIELD8, J43.SHIELD9
- new net SWDCLK1: J22.3, U10.45
- new net SWDCLK2: J36.3, U17.45
- new net SWDCLK3: J50.3, U24.45
- new net SWDIO1: J22.4, U10.46
- new net SWDIO2: J36.4, U17.46
- new net SWDIO3: J50.4, U24.46
- new net TXO1: J19.9, U10.15
- new net TXO2: J33.9, U17.15
- new net TXO3: J47.9, U24.15
- new net TX_LED1: R18.1, U10.39
- new net TX_LED2: R31.1, U17.39
- new net TX_LED3: R44.1, U24.39
- new net USB_VCC1: C17.2, C21.1, D7.A, F2.2, J14.VBUS, J17.2, JP2.2, U2.4
- new net USB_VCC2: C32.2, C36.1, D12.A, F3.2, J29.VBUS, J31.2, JP3.2, U15.4
- new net USB_VCC3: C47.2, C51.1, D17.A, F4.2, J43.VBUS, J45.2, JP4.2, U22.4
- new net VBATT1: C16.+, J16.2, J28.VIN0, R20.2, S2.3, U2.3
- new net VBATT2: C31.+, J30.2, J42.VIN0, R33.2, S5.3, U15.3
- new net VBATT3: C46.+, J44.2, J56.VIN0, R46.2, S7.3, U22.3
- new net VBATT_LVL1: R20.1, R21.2, U10.47
- new net VBATT_LVL2: R33.1, R34.2, U17.47
- new net VBATT_LVL3: R46.1, R47.2, U24.47
- new net VDDANA1: C26.2, L2.2, U10.6
- new net VDDANA2: C41.2, L3.2, U17.6
- new net VDDANA3: C56.2, L4.2, U24.6
Routing:
- net 3.3V2: track 0.00 -> 187.3 mm, vias 0 -> 13
- net 3.3V1: track 0.00 -> 187.3 mm, vias 0 -> 13
- net 3.3V3: track 0.00 -> 187.3 mm, vias 0 -> 13
- net GND3: track 0.00 -> 138.2 mm, vias 0 -> 27
- net GND2: track 0.00 -> 138.2 mm, vias 0 -> 27
- net GND1: track 0.00 -> 138.2 mm, vias 0 -> 27
- net USB_VCC3: track 0.00 -> 100.4 mm, vias 0 -> 6
- net USB_VCC2: track 0.00 -> 100.4 mm, vias 0 -> 6
- net USB_VCC1: track 0.00 -> 100.4 mm, vias 0 -> 6
- net MISO3: track 0.00 -> 83.7 mm, vias 0 -> 5
- net MISO1: track 0.00 -> 83.7 mm, vias 0 -> 5
- net MISO2: track 0.00 -> 83.7 mm, vias 0 -> 5
- net !RST3: track 0.00 -> 83.3 mm, vias 0 -> 5
- net !RST1: track 0.00 -> 83.3 mm, vias 0 -> 5
- net !RST2: track 0.00 -> 83.3 mm, vias 0 -> 5
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- added copper zone on layer 1, net ANT1
- added copper zone on layer 16, net ANT1
- added copper zone on layer 1, net ANT2
- added copper zone on layer 16, net ANT2
- added copper zone on layer 1, net ANT3
- added copper zone on layer 16, net ANT3
- added copper zone on layer 1, net GND1
- added copper zone on layer 16, net GND1
- added copper zone on layer 1, net GND2
- added copper zone on layer 16, net GND2
- added copper zone on layer 1, net GND3
- added copper zone on layer 16, net GND3
- added copper zone on layer 1, net SHLD1
- added copper zone on layer 16, net SHLD1
- added copper zone on layer 1, net SHLD2
- added copper zone on layer 16, net SHLD2
- added copper zone on layer 1, net SHLD3
- added copper zone on layer 16, net SHLD3
Other:
- board size 53.3 x 40.6 mm -> 134.9 x 95.5 mm
- board text added: "Route Out"
- board text added: "v-score"
- board text removed: "0.8mm Board Thickness"
- board text removed: "Owen Lyke"

Commit message: x02 ready for order
Parts:
- removed J53: U.FL, SparkFun-Connectors:U.FL
- removed J54, J55: (no value), SparkFun-Connectors:1X04_1MM_RA
- removed J56: 5.5x2.1mm Barrel, SparkFun-Connectors:POWER_JACK_SMD
- removed LED1, LED2, LED3: RED, SparkFun-LED:LED-0603
- removed LOGO1, LOGO2, LOGO3, LOGO4: OSHW-LOGOMINI, SparkFun-Aesthetics:OSHW-LOGO-MINI
- removed U25: ADJ5, SparkFun-IC-Power:SOT223
- removed U26: E19-915MS1W, SAMD21_ProRF_1W:E19-915MS1W
- removed U27: TXB0108DQSR, SparkFun-IC-Comms:UFDFN-20
- removed U28: 3.3V, SparkFun-IC-Power:SOT23-5
- added D22, D23: 3A/10V/300mV, SAMD21_ProRF_1W:SOD-323
- added D24: BLUE, SparkFun-LED:LED-0603
- added Q5, Q6, Q7, Q8: 310mA/60V/1.6Ω, SparkFun-DiscreteSemi:SOT323
- added R53: 10k, SparkFun-Resistors:0603
- added R54: 1k, SparkFun-Resistors:0603
- added R55, R56: 2.2k, SparkFun-Resistors:0603
- added U$261: (no value), buzzard_labels:SPI11
- added U$262: (no value), buzzard_labels:MISO17
- added U$263: (no value), buzzard_labels:MOSI16
- added U$264: (no value), buzzard_labels:SCK18
- added U$265, U$266: (no value), Labels:QWIIC_COPYRIGHT_SMALL
- added U$267, U$268: (no value), Labels:QWIIC_COPYRIGHT_MEDIUM
- C1: value 10uF -> 15pF; device SparkFun-Capacitors:EIA3216 -> SparkFun-Capacitors:0603
- C10: value 0.1uF -> 10uF; device SparkFun-Capacitors:0603 -> SparkFun-Capacitors:EIA3216
- C11, C14: value 0.1uF -> 1.0uF
- C12: value 1.0uF -> 10uF; device SparkFun-Capacitors:0603 -> SparkFun-Capacitors:EIA3216
- C13, C7: value 10uF -> 0.1uF; device SparkFun-Capacitors:EIA3216 -> SparkFun-Capacitors:0603
- C3: value 15pF -> 0.1uF
- C5: value 1.0uF -> 0.1uF
- C8: value 0.1uF -> 4.7uF
- C9: value 4.7uF -> 10uF; device SparkFun-Capacitors:0603 -> SparkFun-Capacitors:EIA3216
- D1: value Green -> Yellow
- D11, D16: value Green -> 3A/10V/300mV; device SparkFun-LED:LED-0603 -> SAMD21_ProRF_1W:SOD-323
- D13: value Yellow -> Green
- D14, D20: value 3A/10V/300mV -> Yellow; device SAMD21_ProRF_1W:SOD-323 -> SparkFun-LED:LED-0603
- D15, D9: value 3A/10V/300mV -> RED; device SAMD21_ProRF_1W:SOD-323 -> SparkFun-LED:LED-0603
- D17, D4: value BLUE -> 3A/10V/300mV; device SparkFun-LED:LED-0603 -> SAMD21_ProRF_1W:SOD-323
- D18: value Yellow -> BLUE
- D19: value 3A/10V/300mV -> Green; device SAMD21_ProRF_1W:SOD-323 -> SparkFun-LED:LED-0603
- D3: value 3A/10V/300mV -> BLUE; device SAMD21_ProRF_1W:SOD-323 -> SparkFun-LED:LED-0603
- D6: value Yellow -> RED
- D7: value BLUE -> Green
- J10: value AVR_SPI_PROG_3X2TESTPOINTS -> (none); device SparkFun-Connectors:2X3_TEST_POINTS -> SparkFun-Connectors:1X10_NO_SILK
- J11, J23, J37, J49: device SparkFun-Connectors:1X09_NO_SILK -> SparkFun-Connectors:1X04_1MM_RA
- J12: value 5.5x2.1mm Barrel -> (none); device SparkFun-Connectors:POWER_JACK_SMD -> SparkFun-Connectors:1X01_NO_SILK
- J13: value U.FL -> (none); device SparkFun-Connectors:U.FL -> SparkFun-Connectors:1X04_1MM_RA
- J14: value (none) -> CORTEX_DEBUG_PTH; device SparkFun-Connectors:USB-MICROB-PTH-MILL -> SparkFun-Connectors:2X5-PTH-1.27MM
- J15, J41: value (none) -> PTH; device SparkFun-Connectors:1X04_1MM_RA -> SparkFun-Connectors:1X02_NO_SILK
- J16: value PTH -> (none)
- J17, J8: value (none) -> External On/Off
- J18, J32: value External On/Off -> (none); device SparkFun-Connectors:1X02_NO_SILK -> SparkFun-Connectors:1X10_NO_SILK
- J2, J27, J40: device SparkFun-Connectors:1X04_1MM_RA -> SparkFun-Connectors:USB-MICROB-PTH-MILL
- J20, J33, J34, J47: device SparkFun-Connectors:1X10_NO_SILK -> SparkFun-Connectors:1X09_NO_SILK
- J22: value AVR_SPI_PROG_3X2TESTPOINTS -> (none); device SparkFun-Connectors:2X3_TEST_POINTS -> SparkFun-Connectors:1X01_NO_SILK
- J24: device SparkFun-Connectors:1X01_NO_SILK -> SparkFun-Connectors:1X04_1MM_RA
- J25: value U.FL -> 5.5x2.1mm Barrel; device SparkFun-Connectors:U.FL -> SparkFun-Connectors:POWER_JACK_SMD
- J26: value (none) -> CORTEX_DEBUG_PTH; device SparkFun-Connectors:1X04_1MM_RA -> SparkFun-Connectors:2X5-PTH-1.27MM
- J28: value 5.5x2.1mm Barrel -> PTH; device SparkFun-Connectors:POWER_JACK_SMD -> SparkFun-Connectors:1X02_NO_SILK
- J29: device SparkFun-Connectors:USB-MICROB-PTH-MILL -> SparkFun-Connectors:1X02_NO_SILK
- J3: value (none) -> PTH; device SparkFun-Connectors:1X10_NO_SILK -> SparkFun-Connectors:1X02_NO_SILK
- J30: value PTH -> External On/Off
- J31, J45: device SparkFun-Connectors:1X02_NO_SILK -> SparkFun-Connectors:1X10_NO_SILK
- J35: device SparkFun-Connectors:1X09_NO_SILK -> SparkFun-Connectors:1X01_NO_SILK
- J36, J50: value AVR_SPI_PROG_3X2TESTPOINTS -> (none); device SparkFun-Connectors:2X3_TEST_POINTS -> SparkFun-Connectors:1X04_1MM_RA
- J38: value (none) -> 5.5x2.1mm Barrel; device SparkFun-Connectors:1X01_NO_SILK -> SparkFun-Connectors:POWER_JACK_SMD
- J39: value U.FL -> CORTEX_DEBUG_PTH; device SparkFun-Connectors:U.FL -> SparkFun-Connectors:2X5-PTH-1.27MM
- J4: device SparkFun-Connectors:1X01_NO_SILK -> SparkFun-Connectors:1X02_NO_SILK
- J42: value 5.5x2.1mm Barrel -> (none); device SparkFun-Connectors:POWER_JACK_SMD -> SparkFun-Connectors:1X02_NO_SILK
- J43: value (none) -> External On/Off; device SparkFun-Connectors:USB-MICROB-PTH-MILL -> SparkFun-Connectors:1X02_NO_SILK
- J44: value PTH -> (none); device SparkFun-Connectors:1X02_NO_SILK -> SparkFun-Connectors:1X10_NO_SILK
- J46, J9: value External On/Off -> (none); device SparkFun-Connectors:1X02_NO_SILK -> SparkFun-Connectors:1X09_NO_SILK
- J48: device SparkFun-Connectors:1X10_NO_SILK -> SparkFun-Connectors:1X01_NO_SILK
- J5, J51: value (none) -> 5.5x2.1mm Barrel; device SparkFun-Connectors:1X09_NO_SILK -> SparkFun-Connectors:POWER_JACK_SMD
- J52: value (none) -> CORTEX_DEBUG_PTH; device SparkFun-Connectors:1X01_NO_SILK -> SparkFun-Connectors:2X5-PTH-1.27MM
- J7: value PTH -> (none); device SparkFun-Connectors:1X02_NO_SILK -> SparkFun-Connectors:1X09_NO_SILK
- R10, R19, R31, R45, R7, R9: value 1k -> 10k
- R11: value 2.0k -> 10k
- R13, R27, R28, R41: value 1k -> 2.2k
- R14: value 750K -> 2.2k
- R15: value 240 -> 1k
- R16, R2, R26, R30, R43, R46, R8: value 10k -> 1k
- R20, R34, R48, R6: value 10k -> 750
- R21, R35: value 10k -> 240
- R23, R36: value 750K -> 10k
- R24, R37, R50: value 240 -> 10k
- R29: value 2.0k -> 1k
- R42: value 2.0k -> 2.2k
- R49: value 750K -> 240
- R5: value 2.0k -> 240
- S1: value Power -> MOMENTARY-SWITCH-SPST-SMD-5.2-REDUNDANT; device SparkFun-Switches:SWITCH_SPST_SMD_A -> SparkFun-Switches:TACTILE_SWITCH_SMD_5.2MM
- S3: value (none) -> Power; device SparkFun-Switches:TACTILE_SWITCH_SMD_RIGHT_ANGLE -> SparkFun-Switches:SWITCH_SPST_SMD_A
- S4, S6, S8: value (none) -> MOMENTARY-SWITCH-SPST-SMD-5.2-REDUNDANT; device SparkFun-Switches:TACTILE_SWITCH_SMD_RIGHT_ANGLE -> SparkFun-Switches:TACTILE_SWITCH_SMD_5.2MM
- U$10: device buzzard_labels (25):SCK10 -> buzzard_labels:MISO4
- U$100: device buzzard_labels (8):RX7 -> buzzard_labels (10):D90
- U$101: device buzzard_labels (8):RX2 -> buzzard_labels (10):D90
- U$102: device buzzard_labels (9):CHG1 -> buzzard_labels (25):GND0
- U$103: device buzzard_labels (25):D514 -> buzzard_labels (8):RX2
- U$104: device buzzard_labels (10):D90 -> buzzard_labels (8):TX3
- U$105: device buzzard_labels (10):D90 -> D5:D50
- U$106: device buzzard_labels (25):GND0 -> SparkFun-Aesthetics:OSHW-LOGO-MINI
- U$107: device buzzard_labels (8):RX2 -> buzzard_labels:SAMD21_PRORF_1W5
- U$108: device buzzard_labels (8):TX3 -> buzzard_labels:VUSB7
- U$109, U$243: device D2:D20 -> buzzard_labels:VUSB7
- U$110, U$244: device D3:D30 -> buzzard_labels:SWITCH6
- U$111, U$245: device D4:D40 -> buzzard_labels:SWITCH6
- U$112: device D5:D50 -> buzzard_labels:7#15V0
- U$113: device D2:D20 -> buzzard_labels:SOLDER_TO_BYPASS_VUSB_FUSE1
- U$114: value (none) -> SPARKX-LOGO4; device D3:D30 -> SparkX:SPARKX-MEDIUM
- U$115, U$241: device D4:D40 -> buzzard_labels:SAMD21_PRORF_1W5
- U$116: value SPARKX-LOGO2 -> (none); device SparkX:SPARKX-TINY -> SparkX:SPARKX-MEDIUM
- U$117: device Labels:QWIIC-LOGO-MEDIUM -> buzzard_labels:D130
- U$118: device SparkX:SPARKX-MEDIUM -> buzzard_labels:OFF#ON1
- U$119: device SparkFun-Aesthetics:OSHW-LOGO-MINI -> buzzard_labels:SPI2
- U$120: device buzzard_labels:SAMD21_PRORF_1W5 -> buzzard_labels:MOSI3
- U$121: device buzzard_labels:VUSB7 -> buzzard_labels:MISO4
- U$122: device buzzard_labels:VUSB7 -> buzzard_labels:SCK5
- U$123, U$188: device buzzard_labels:SWITCH6 -> buzzard_labels:MISO4
- U$124, U$189: device buzzard_labels:SWITCH6 -> buzzard_labels:SCK5
- U$125, U$259: device Labels:QWIIC-TEXT-04 -> buzzard_labels:MOSI3
- U$126, U$194, U$260: device Labels:QWIIC-TEXT-04 -> buzzard_labels:SPI11
- U$127: device buzzard_labels:7#15V0 -> buzzard_labels:SPI11
- U$128: device buzzard_labels:SOLDER_TO_BYPASS_VUSB_FUSE1 -> buzzard_labels:MISO17
- U$129: device Labels:QWIIC-TEXT-04 -> buzzard_labels:MOSI16
- U$130: device Labels:QWIIC-TEXT-04 -> buzzard_labels:SCK18
- U$131: device buzzard_labels (25):A43 -> Labels:QWIIC_COPYRIGHT_SMALL
- U$132: device buzzard_labels (25):A34 -> Labels:QWIIC_COPYRIGHT_SMALL
- U$133: device buzzard_labels (25):A25 -> Labels:QWIIC_COPYRIGHT_MEDIUM
- U$134: device buzzard_labels (25):A16 -> Labels:QWIIC_COPYRIGHT_MEDIUM
- U$135: device buzzard_labels (25):A07 -> buzzard_labels (25):A43
- U$136: device buzzard_labels (25):MISO8 -> buzzard_labels (25):A34
- U$137: device buzzard_labels (25):MOSI9 -> buzzard_labels (25):A25
- U$138: device buzzard_labels (25):SCK10 -> buzzard_labels (25):A16
- U$139: device buzzard_labels (25):ANT11 -> buzzard_labels (25):A07
- U$140: device buzzard_labels (25):GND0 -> buzzard_labels (25):ANT11
- U$141, U$214: device buzzard_labels (25):RST2 -> buzzard_labels (25):GND0
- U$142: device buzzard_labels (25):3V320 -> buzzard_labels (25):RST2
- U$143, U$159: device buzzard_labels (25):RAW21 -> buzzard_labels (25):3V320
- U$144, U$211: device buzzard_labels (25):RST2 -> buzzard_labels (25):RAW21
- U$145: device buzzard_labels (25):BATT25 -> buzzard_labels (25):RST2
- U$146, U$78: device buzzard_labels (25):RST2 -> buzzard_labels (25):BATT25
- U$148: device buzzard_labels (28):ON#OFF0 -> buzzard_labels (25):RST2
- U$149: device buzzard_labels (25):RST2 -> buzzard_labels (25):A43
- U$150: device buzzard_labels (25):A43 -> buzzard_labels (25):A34
- U$151: device buzzard_labels (25):A34 -> buzzard_labels (25):A25
- U$152: device buzzard_labels (25):A25 -> buzzard_labels (25):A16
- U$153: device buzzard_labels (25):A16 -> buzzard_labels (25):A07
- U$154: device buzzard_labels (25):A07 -> buzzard_labels (25):MISO8
- U$155: device buzzard_labels (25):MISO8 -> buzzard_labels (25):MOSI9
- U$156: device buzzard_labels (25):MOSI9 -> buzzard_labels (25):SCK10
- U$157, U$68: device buzzard_labels (25):SCK10 -> buzzard_labels (25):ANT11
- U$158: device buzzard_labels (25):ANT11 -> buzzard_labels (25):RAW21
- U$160: device buzzard_labels (25):3V320 -> buzzard_labels (25):GND0
- U$161: device buzzard_labels (25):GND0 -> Labels:PWR-()-03
- U$162: device Labels:PWR-()-03 -> buzzard_labels (8):TX3
- U$163: device buzzard_labels (8):TX3 -> buzzard_labels (8):TX6
- U$164: device buzzard_labels (8):TX6 -> buzzard_labels (8):RX7
- U$165: device buzzard_labels (8):RX7 -> buzzard_labels (8):RX2
- U$166: device buzzard_labels (8):RX2 -> buzzard_labels (25):D514
- U$167: device buzzard_labels (9):CHG1 -> buzzard_labels (10):D90
- U$168: device buzzard_labels (25):D514 -> buzzard_labels (10):D90
- U$169: device buzzard_labels (10):D90 -> buzzard_labels (25):GND0
- U$170: device buzzard_labels (10):D90 -> buzzard_labels (8):RX2
- U$171: device buzzard_labels (25):GND0 -> buzzard_labels (8):TX3
- U$172: device buzzard_labels (8):RX2 -> D5:D50
- U$173: device buzzard_labels (8):TX3 -> SparkFun-Aesthetics:OSHW-LOGO-MINI
- U$174: device D2:D20 -> buzzard_labels:SAMD21_PRORF_1W5
- U$175: device D3:D30 -> buzzard_labels:VUSB7
- U$176: device D4:D40 -> buzzard_labels:VUSB7
- U$177: device D5:D50 -> buzzard_labels:SWITCH6
- U$178: device D2:D20 -> buzzard_labels:SWITCH6
- U$179: device D3:D30 -> buzzard_labels:7#15V0
- U$18: device D2:D20 -> buzzard_labels:SCK5
- U$180: device D4:D40 -> buzzard_labels:SOLDER_TO_BYPASS_VUSB_FUSE1
- U$181, U$34: value SPARKX-LOGO2 -> SPARKX-LOGO4; device SparkX:SPARKX-TINY -> SparkX:SPARKX-MEDIUM
- U$182: device Labels:QWIIC-LOGO-MEDIUM -> buzzard_labels:SAMD21_PRORF_1W5
- U$184: device SparkFun-Aesthetics:OSHW-LOGO-MINI -> buzzard_labels:D130
- U$185: device buzzard_labels:SAMD21_PRORF_1W5 -> buzzard_labels:OFF#ON1
- U$186: device buzzard_labels:VUSB7 -> buzzard_labels:SPI2
- U$187: device buzzard_labels:VUSB7 -> buzzard_labels:MOSI3
- U$190, U$255: device Labels:QWIIC-TEXT-04 -> buzzard_labels:MISO4
- U$191, U$256: device Labels:QWIIC-TEXT-04 -> buzzard_labels:SCK5
- U$192: device buzzard_labels:7#15V0 -> buzzard_labels:MOSI3
- U$193: device buzzard_labels:SOLDER_TO_BYPASS_VUSB_FUSE1 -> buzzard_labels:SPI11
- U$195: device Labels:QWIIC-TEXT-04 -> buzzard_labels:MISO17
- U$196: device buzzard_labels (25):A43 -> buzzard_labels:MOSI16
- U$197: device buzzard_labels (25):A34 -> buzzard_labels:SCK18
- U$198: device buzzard_labels (25):A25 -> Labels:QWIIC_COPYRIGHT_SMALL
- U$199: device buzzard_labels (25):A16 -> Labels:QWIIC_COPYRIGHT_SMALL
- U$2: device D2:D20 -> buzzard_labels:MISO4
- U$20: device D3:D30 -> buzzard_labels:MOSI3
- U$200: device buzzard_labels (25):A07 -> Labels:QWIIC_COPYRIGHT_MEDIUM
- U$201: device buzzard_labels (25):MISO8 -> Labels:QWIIC_COPYRIGHT_MEDIUM
- U$202: device buzzard_labels (25):MOSI9 -> buzzard_labels (25):A43
- U$203: device buzzard_labels (25):SCK10 -> buzzard_labels (25):A34
- U$204: device buzzard_labels (25):ANT11 -> buzzard_labels (25):A25
- U$205: device buzzard_labels (25):GND0 -> buzzard_labels (25):A16
- U$206: device buzzard_labels (25):RST2 -> buzzard_labels (25):A07
- U$207: device buzzard_labels (25):3V320 -> buzzard_labels (25):ANT11
- U$208: device buzzard_labels (25):RAW21 -> buzzard_labels (25):GND0
- U$21: device D3:D30 -> buzzard_labels:SPI11
- U$210: device buzzard_labels (25):BATT25 -> buzzard_labels (25):3V320
- U$212, U$74: device buzzard_labels (25):GND0 -> buzzard_labels (25):RST2
- U$213: device buzzard_labels (28):ON#OFF0 -> buzzard_labels (25):BATT25
- U$215: device buzzard_labels (25):A43 -> buzzard_labels (25):RST2
- U$216: device buzzard_labels (25):A34 -> buzzard_labels (25):A43
- U$217: device buzzard_labels (25):A25 -> buzzard_labels (25):A34
- U$218: device buzzard_labels (25):A16 -> buzzard_labels (25):A25
- U$219: device buzzard_labels (25):A07 -> buzzard_labels (25):A16
- U$22: device D4:D40 -> buzzard_labels:MISO17
- U$220, U$66: device buzzard_labels (25):MISO8 -> buzzard_labels (25):A07
- U$221: device buzzard_labels (25):MOSI9 -> buzzard_labels (25):MISO8
- U$222: device buzzard_labels (25):SCK10 -> buzzard_labels (25):MOSI9
- U$223: device buzzard_labels (25):ANT11 -> buzzard_labels (25):SCK10
- U$224: device buzzard_labels (25):RAW21 -> buzzard_labels (25):ANT11
- U$225, U$76: device buzzard_labels (25):3V320 -> buzzard_labels (25):RAW21
- U$226: device buzzard_labels (25):GND0 -> buzzard_labels (25):3V320
- U$227: device Labels:PWR-()-03 -> buzzard_labels (25):GND0
- U$228: device buzzard_labels (8):TX3 -> Labels:PWR-()-03
- U$229: device buzzard_labels (8):TX6 -> buzzard_labels (8):TX3
- U$230: device buzzard_labels (8):RX7 -> buzzard_labels (8):TX6
- U$231: device buzzard_labels (8):RX2 -> buzzard_labels (8):RX7
- U$232: device buzzard_labels (9):CHG1 -> buzzard_labels (8):RX2
- U$239: device D2:D20 -> D5:D50
- U$240: device D3:D30 -> SparkFun-Aesthetics:OSHW-LOGO-MINI
- U$242: device D5:D50 -> buzzard_labels:VUSB7
- U$246: value SPARKX-LOGO2 -> (none); device SparkX:SPARKX-TINY -> buzzard_labels:7#15V0
- U$247: device Labels:QWIIC-LOGO-MEDIUM -> buzzard_labels:SOLDER_TO_BYPASS_VUSB_FUSE1
- U$248: value (none) -> SPARKX-LOGO4
- U$249: device SparkFun-Aesthetics:OSHW-LOGO-MINI -> buzzard_labels:SAMD21_PRORF_1W5
- U$250: device buzzard_labels:SAMD21_PRORF_1W5 -> SparkX:SPARKX-MEDIUM
- U$251: device buzzard_labels:VUSB7 -> buzzard_labels:D130
- U$252: device buzzard_labels:VUSB7 -> buzzard_labels:OFF#ON1
- U$253: device buzzard_labels:SWITCH6 -> buzzard_labels:SPI2
- U$254: device buzzard_labels:SWITCH6 -> buzzard_labels:MOSI3
- U$257: device buzzard_labels:7#15V0 -> buzzard_labels:MISO4
- U$258: device buzzard_labels:SOLDER_TO_BYPASS_VUSB_FUSE1 -> buzzard_labels:SCK5
- U$26: device buzzard_labels (25):A43 -> buzzard_labels:SAMD21_PRORF_1W5
- U$29: device Labels:QWIIC-TEXT-04 -> buzzard_labels (25):A43
- U$30: device Labels:QWIIC-LOGO-MEDIUM -> Labels:QWIIC_COPYRIGHT_MEDIUM
- U$31: device D4:D40 -> buzzard_labels:MOSI16
- U$36: device buzzard_labels (25):RST2 -> buzzard_labels:OFF#ON1
- U$39: device buzzard_labels (28):ON#OFF0 -> buzzard_labels:SCK5
- U$40: device Labels:QWIIC-TEXT-04 -> buzzard_labels (25):A34
- U$51: device SparkX:SPARKX-MEDIUM -> Labels:QWIIC_COPYRIGHT_MEDIUM
- U$54: device Labels:QWIIC-TEXT-04 -> buzzard_labels (25):A25
- U$56: device Labels:QWIIC-TEXT-04 -> buzzard_labels (25):A16
- U$58: device buzzard_labels (25):A34 -> SparkX:SPARKX-MEDIUM
- U$59: device buzzard_labels (25):A25 -> buzzard_labels:D130
- U$60: device buzzard_labels (25):A16 -> buzzard_labels:SCK18
- U$64: device buzzard_labels (25):A07 -> Labels:QWIIC_COPYRIGHT_SMALL
- U$65: device buzzard_labels (9):CHG1 -> buzzard_labels:SPI11
- U$67: device buzzard_labels (25):MOSI9 -> Labels:QWIIC_COPYRIGHT_SMALL
- U$71, U$93: device buzzard_labels (25):ANT11 -> buzzard_labels (25):GND0
- U$75: device buzzard_labels (25):RST2 -> buzzard_labels (25):3V320
- U$77: device buzzard_labels (25):RAW21 -> buzzard_labels (25):RST2
- U$79: device buzzard_labels (25):BATT25 -> buzzard_labels (25):GND0
- U$8: device buzzard_labels (25):MISO8 -> buzzard_labels:SPI2
- U$82: device buzzard_labels (25):GND0 -> buzzard_labels (25):A43
- U$83: device buzzard_labels (28):ON#OFF0 -> buzzard_labels (25):A34
- U$84: device buzzard_labels (25):RST2 -> buzzard_labels (25):A25
- U$85: device buzzard_labels (25):A43 -> buzzard_labels (25):A16
- U$86: device buzzard_labels (25):A34 -> buzzard_labels (25):A07
- U$87: device buzzard_labels (25):A25 -> buzzard_labels (25):MISO8
- U$88: device buzzard_labels (25):A16 -> buzzard_labels (25):MOSI9
- U$89: device buzzard_labels (25):A07 -> buzzard_labels (25):SCK10
- U$9: device buzzard_labels (25):MOSI9 -> buzzard_labels:MOSI3
- U$90: device buzzard_labels (25):MISO8 -> buzzard_labels (25):ANT11
- U$91: device buzzard_labels (25):MOSI9 -> buzzard_labels (25):RAW21
- U$92: device buzzard_labels (25):SCK10 -> buzzard_labels (25):3V320
- U$94: device buzzard_labels (25):RAW21 -> Labels:PWR-()-03
- U$95: device buzzard_labels (25):3V320 -> buzzard_labels (8):TX3
- U$96: device buzzard_labels (25):GND0 -> buzzard_labels (8):TX6
- U$97: device Labels:PWR-()-03 -> buzzard_labels (8):RX7
- U$98: device buzzard_labels (8):TX3 -> buzzard_labels (8):RX2
- U$99: device buzzard_labels (8):TX6 -> buzzard_labels (25):D514
- U1: value MCP73831 -> ATSAMD21G; device SparkFun-IC-Power:SOT23-5 -> temp:QFN-48_NO_EXPOSED_PAD
- U10: value ATSAMD21G -> E19-915MS1W; device temp:QFN-48_NO_EXPOSED_PAD -> SAMD21_ProRF_1W:E19-915MS1W
- U11: value ADJ5 -> TXB0108DQSR; device SparkFun-IC-Power:SOT223 -> SparkFun-IC-Comms:UFDFN-20
- U12: value E19-915MS1W -> 3.3V; device SAMD21_ProRF_1W:E19-915MS1W -> SparkFun-IC-Power:SOT23-5
- U13: value TXB0108DQSR -> 4MB Flash; device SparkFun-IC-Comms:UFDFN-20 -> SparkFun-IC-Memory:SO08
- U14: value 3.3V -> ATSAMD21G; device SparkFun-IC-Power:SOT23-5 -> temp:QFN-48_NO_EXPOSED_PAD
- U15: value MCP73831 -> ADJ5; device SparkFun-IC-Power:SOT23-5 -> SparkFun-IC-Power:SOT223
- U16, U5: value 4MB Flash -> E19-915MS1W; device SparkFun-IC-Memory:SO08 -> SAMD21_ProRF_1W:E19-915MS1W
- U17: value ATSAMD21G -> TXB0108DQSR; device temp:QFN-48_NO_EXPOSED_PAD -> SparkFun-IC-Comms:UFDFN-20
- U18: value ADJ5 -> 3.3V; device SparkFun-IC-Power:SOT223 -> SparkFun-IC-Power:SOT23-5
- U19: value E19-915MS1W -> 4MB Flash; device SAMD21_ProRF_1W:E19-915MS1W -> SparkFun-IC-Memory:SO08
- U2: value MCP73831 -> 3.3V
- U20, U8: value TXB0108DQSR -> ATSAMD21G; device SparkFun-IC-Comms:UFDFN-20 -> temp:QFN-48_NO_EXPOSED_PAD
- U21, U3: value 3.3V -> ADJ5; device SparkFun-IC-Power:SOT23-5 -> SparkFun-IC-Power:SOT223
- U22: value MCP73831 -> E19-915MS1W; device SparkFun-IC-Power:SOT23-5 -> SAMD21_ProRF_1W:E19-915MS1W
- U23: value 4MB Flash -> TXB0108DQSR; device SparkFun-IC-Memory:SO08 -> SparkFun-IC-Comms:UFDFN-20
- U24: value ATSAMD21G -> 3.3V; device temp:QFN-48_NO_EXPOSED_PAD -> SparkFun-IC-Power:SOT23-5
- U4: value ATSAMD21G -> 4MB Flash; device temp:QFN-48_NO_EXPOSED_PAD -> SparkFun-IC-Memory:SO08
- U6: value E19-915MS1W -> TXB0108DQSR; device SAMD21_ProRF_1W:E19-915MS1W -> SparkFun-IC-Comms:UFDFN-20
- U7: value ADJ5 -> 4MB Flash; device SparkFun-IC-Power:SOT223 -> SparkFun-IC-Memory:SO08
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- renumbered LED4 to D21
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Connections:
- removed net !RFM_CS: Q1.2, R12.1, U4.28
- removed net !RFM_CS1: Q2.2, R25.1, U10.28
- removed net !RFM_CS2: Q3.2, R38.1, U17.28
- removed net !RFM_CS3: Q4.2, R51.1, U24.28
- removed net !RFM_CS5V: Q1.3, R16.1, U6.P$15
- removed net !RFM_CS5V1: Q2.3, R26.1, U12.P$15
- removed net !RFM_CS5V2: Q3.3, R39.1, U19.P$15
- removed net !RFM_CS5V3: Q4.3, R52.1, U26.P$15
- removed net CHARGE_STAT: R9.1, U1.1
- removed net CHARGE_STAT1: R19.1, U2.1
- removed net CHARGE_STAT2: R32.1, U15.1
- removed net CHARGE_STAT3: R45.1, U22.1
- removed net D21: J33.3, U17.12
- removed net D22: J47.4, U24.13
- removed net D23: U24.27, U27.9
- removed net D24: U24.25, U27.10
- removed net D25: J47.6, U24.23
- removed net D26: J47.5, U24.14
- removed net D27: J47.7, U24.24
- removed net D28: J47.3, U24.12
- removed net N$36: D21.A, R41.1
- removed net N$37: D18.C, R40.2
- removed net N$39: D16.C, R44.2
- removed net N$40: C52.2, U24.1, Y4.P$2
- removed net N$41: C53.2, U24.2, Y4.P$1
- removed net N$42: R49.2, R50.1, U25.1
- removed net N$43: D19.A, F4.1, JP4.1
- removed net N$44: D20.A, R50.2, U25.2, U25.4
- removed net RFM_INT: U4.29, U8.8
- removed net RFM_INT1: U10.29, U13.8
- removed net RFM_INT2: U17.29, U20.8
- removed net RFM_INT3: U24.29, U27.8
- removed net RFM_RST: U4.26, U6.P$8
- removed net RFM_RST1: U10.26, U12.P$8
- removed net RFM_RST2: U17.26, U19.P$8
- removed net RFM_RST3: U24.26, U26.P$8
- removed net RFM_RXEN: U4.38, U8.7
- removed net RFM_RXEN1: U10.38, U13.7
- removed net RFM_RXEN2: U17.38, U20.7
- removed net RFM_RXEN3: U24.38, U27.7
- removed net RFM_RXEN5V: U6.P$17, U8.14
- removed net RFM_RXEN5V1: U12.P$17, U13.14
- removed net RFM_RXEN5V2: U19.P$17, U20.14
- removed net RFM_RXEN5V3: U26.P$17, U27.14
- removed net RFM_TXEN: U4.37, U8.4
- removed net RFM_TXEN1: U10.37, U13.4
- removed net RFM_TXEN2: U17.37, U20.4
- removed net RFM_TXEN3: U24.37, U27.4
- removed net RFM_TXEN5V: U6.P$16, U8.17
- removed net RFM_TXEN5V1: U12.P$16, U13.17
- removed net RFM_TXEN5V2: U19.P$16, U20.17
- removed net RFM_TXEN5V3: U26.P$16, U27.17
- removed net VBATT_LVL: R1.1, R2.2, U4.47
- removed net VBATT_LVL1: R20.1, R21.2, U10.47
- removed net VBATT_LVL2: R33.1, R34.2, U17.47
- removed net VBATT_LVL3: R46.1, R47.2, U24.47
- new net !E19_CS: Q2.2, R10.1, U1.28
- new net !E19_CS1: Q3.2, R22.1, U8.28
- new net !E19_CS2: Q5.2, R36.1, U14.28
- new net !E19_CS3: Q7.2, R50.1, U20.28
- new net !E19_CS5V: Q2.3, R12.1, U5.P$15
- new net !E19_CS5V1: Q3.3, R23.1, U10.P$15
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Routing:
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- removed copper zone on layer 1, net ANT
- removed copper zone on layer 1, net ANT1
- removed copper zone on layer 1, net ANT2
- removed copper zone on layer 1, net ANT3
Other:
- board text added: "Owen Lyke"
- board text added: "x02"
- board text removed: "x01"
